File: max232_conv.kicad_pcb (KiCad board)
At the start: 2 copper layers, 99.5 x 49.9 mm, 21 parts, among them J1 Conn_01x06, J2 Conn_01x05, J3 Conn_01x06, J4 Conn_01x05, J5 DB9_Male_MountingHoles, U1 MAX232, U2 MAX232

Commit message: Added photo
Parts:
- moved C7 2.35 mm to (168.5, 137.8), turned to 0 degrees
Connections:
- C7 pad 1: Net-(C7-Pad1) -> GND
- C7 pad 2: GND -> Net-(C7-Pad2)
- U2 pad 6: Net-(C7-Pad1) -> Net-(C7-Pad2)
Routing:
- net Net-(C7-Pad2): track 0.00 -> 18.5 mm
- net Net-(C7-Pad1): track 18.5 -> 0.00 mm
Changed lines of the file:
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@@
   (net 42 "Net-(C2-Pad1)")
   (net 43 "Net-(C2-Pad2)")
-  (net 44 "Net-(U1-Pad6)")
+  (net 44 "Net-(C3-Pad2)")
   (net 45 "Net-(C4-Pad1)")
   (net 46 "+5V")
@@
   (net 49 "Net-(C6-Pad1)")
   (net 50 "Net-(C6-Pad2)")
-  (net 51 "Net-(C7-Pad1)")
+  (net 51 "Net-(C7-Pad2)")
   (net 52 "Net-(C8-Pad1)")
   (net 53 "Net-(J1-Pad2)")
@@
   )
   (footprint "Capacitor_THT:CP_Radial_D6.3mm_P2.50mm" (layer "F.Cu")
-    (at 170.815 137.795 180)
+    (at 168.467621 137.75)
     (descr "CP, Radial series, Radial, pin pitch=2.50mm, , diameter=6.3mm, Electrolytic Capacitor")
     (tags "CP Radial series Radial pin pitch 2.50mm  diameter 6.3mm Electrolytic Capacitor")
@@
     (fp_line (start -1.128972 -1.6885) (end -1.128972 -1.0585) (layer "F.Fab") (width 0.1))
     (fp_circle (center 1.25 0) (end 4.4 0) (layer "F.Fab") (width 0.1) (fill none))
-    (pad "1" thru_hole rect (at 0 0 180) (size 1.6 1.6) (drill 0.8) (layers *.Cu *.Mask)
-      (net 51 "Net-(C7-Pad1)") (pintype "passive"))
-    (pad "2" thru_hole circle (at 2.5 0 180) (size 1.6 1.6) (drill 0.8) (layers *.Cu *.Mask)
+    (pad "1" thru_hole rect (at 0 0) (size 1.6 1.6) (drill 0.8) (layers *.Cu *.Mask)
       (net 1 "GND") (pintype "passive"))
+    (pad "2" thru_hole circle (at 2.5 0) (size 1.6 1.6) (drill 0.8) (layers *.Cu *.Mask)
+      (net 51 "Net-(C7-Pad2)") (pintype "passive"))
     (model "${KICAD6_3DMODEL_DIR}/Capacitor_THT.3dshapes/CP_Radial_D6.3mm_P2.50mm.wrl"
       (offset (xyz 0 0 0))
@@
       (net 43 "Net-(C2-Pad2)") (pinfunction "C2-") (pintype "passive"))
     (pad "6" thru_hole oval (at 0 12.7) (size 1.6 1.6) (drill 0.8) (layers *.Cu *.Mask)
-      (net 44 "Net-(U1-Pad6)") (pinfunction "VS-") (pintype "power_out"))
+      (net 44 "Net-(C3-Pad2)") (pinfunction "VS-") (pintype "power_out"))
     (pad "7" thru_hole oval (at 0 15.24) (size 1.6 1.6) (drill 0.8) (layers *.Cu *.Mask)
       (net 59 "Net-(J2-Pad4)") (pinfunction "T2OUT") (pintype "output"))
@@
       (net 50 "Net-(C6-Pad2)") (pinfunction "C2-") (pintype "passive"))
     (pad "6" thru_hole oval (at 0 12.7) (size 1.6 1.6) (drill 0.8) (layers *.Cu *.Mask)
-      (net 51 "Net-(C7-Pad1)") (pinfunction "VS-") (pintype "power_out"))
+      (net 51 "Net-(C7-Pad2)") (pinfunction "VS-") (pintype "power_out"))
     (pad "7" thru_hole oval (at 0 15.24) (size 1.6 1.6) (drill 0.8) (layers *.Cu *.Mask)
       (net 67 "Net-(J4-Pad4)") (pinfunction "T2OUT") (pintype "output"))
@@
       (net 1 "GND") (pintype "passive"))
     (pad "2" thru_hole circle (at 2.5 0) (size 1.6 1.6) (drill 0.8) (layers *.Cu *.Mask)
-      (net 44 "Net-(U1-Pad6)") (pintype "passive"))
+      (net 44 "Net-(C3-Pad2)") (pintype "passive"))
     (model "${KICAD6_3DMODEL_DIR}/Capacitor_THT.3dshapes/CP_Radial_D6.3mm_P2.50mm.wrl"
       (offset (xyz 0 0 0))
